Commit message: 将撼地者添加到gazebo

File: hdz_simplified/urdf/hdz_simplified.urdf (robot description, URDF)
Before this commit: robot hdz_simplified, 2 links, 1 joints
Links:
- link hdz_arm_frame: geometry collision mesh filename=file://$(find hdz_simplified)/meshes/hdz_arm_frame.STL; visual mesh filename=file://$(find hdz_simplified)/meshes/hdz_arm_frame.STL
- link hdz_up_board: geometry collision mesh filename=file://$(find hdz_simplified)/meshes/hdz_up_board.STL; visual mesh filename=file://$(find hdz_simplified)/meshes/hdz_up_board.STL

File: ur_perception_description/urdf/ue5e_perception.urdf.xacro (robot description, xacro)
@@ -1,5 +1,15 @@
 <?xml version="1.0" encoding="UTF-8"?>
 <robot name="ur5e_rgbd" xmlns:xacro="http://www.ros.org/wiki/xacro">
+    <!-- create link fixed to the "world" -->
+    <link name="world" />
+    <!-- 撼地者 -->
+    <xacro:include filename="$(find hdz_simplified)/urdf/hdz_simplified.urdf" />
+    <joint name="hdz_joint" type="fixed">
+        <parent link="world" />
+        <child link="hdz_up_board" />
+        <origin xyz="0.0 0.0 0.487" rpy="0.0 0.0 0.0" />
+    </joint>
     <!-- UR model -->
+    <xacro:arg name="ur_parent" default="hdz_up_board" />
     <xacro:include filename="$(find ur_perception_description)/urdf/ur5e.urdf.xacro" />
     <!-- d435i model -->

File: ur_perception_description/urdf/ur5e.urdf.xacro (robot description, xacro)
@@ -46,14 +46,12 @@
    <xacro:arg name="simulation_controllers" default="" />
    <!-- initial position for simulations (Fake Hardware, Gazebo, Ignition) -->
-   <xacro:arg name="initial_positions_file" default="$(find ur_description)/config/initial_positions.yaml"/>
+   <xacro:arg name="initial_positions_file" default="$(find ur_perception_description)/config/initial_positions.yaml"/>
    <!-- convert to property to use substitution in function -->
    <xacro:property name="initial_positions_file" default="$(arg initial_positions_file)"/>
-   <!-- create link fixed to the "world" -->
-   <link name="world" />
    <!-- arm -->
    <xacro:ur_robot
      name="$(arg name)"
      tf_prefix="$(arg tf_prefix)"
-     parent="world"
+     parent="$(arg ur_parent)"
      joint_limits_parameters_file="$(arg joint_limit_params)"
      kinematics_parameters_file="$(arg kinematics_params)"
@@ -89,5 +87,5 @@
      trajectory_port="$(arg trajectory_port)"
      >
-     <origin xyz="0 0 0.2" rpy="0 0 0" />          <!-- position robot in the world -->
+     <origin xyz="0 -0.3 0.03" rpy="0 0 0" />          <!-- position robot in the world -->
    </xacro:ur_robot>
    <xacro:if value="$(arg sim_gazebo)">

Commit message: 重构 hdz_simplified：generated from solidworks

File: hdz_simplified/urdf/hdz_simplified.urdf (robot description, URDF)
Before this commit: robot hdz_simplified, 2 links, 1 joints
Links:
- removed link hdz_arm_frame
- removed link hdz_up_board
- added link base_frame_link, mass 15.553; collision mesh filename=package://hdz_simplified/meshes/base_frame_link.STL; visual mesh filename=package://hdz_simplified/meshes/base_frame_link.STL
- added link base_link, mass 3.1175; collision mesh filename=package://hdz_simplified/meshes/base_link.STL; visual mesh filename=package://hdz_simplified/meshes/base_link.STL
Joints:
- removed joint hdz_arm_frame_joint
- added joint base_frame_joint: type fixed, parent base_link, child base_frame_link, origin xyz=-0.23005 0 0.005 rpy=0 0 0, axis 0 0 0
