Commit message: update hdz_simplified model

File: hdz_simplified/urdf/hdz_simplified.xacro (robot description, xacro)
@@ -1,66 +1,221 @@
 <?xml version="1.0" encoding="utf-8"?>
-<robot xmlns:xacro="http://www.ros.org/wiki/xacro" name="hdz_simplified">
-  <link name="hdz_base_link" />
-  <link name="hdz_arm_base_link" />
-  <link name="hdz_up_board_link">
-    <inertial>
-      <origin xyz="5.2042E-18 4.4255E-17 0.0025" rpy="0 0 0" />
-      <mass value="3.1175" />
-      <inertia ixx="0.13172" ixy="8.8751E-19" ixz="5.1381E-20"
-        iyy="0.20619" iyz="5.4212E-20" izz="0.3379" />
-    </inertial>
-    <visual>
-      <origin xyz="0 0 0" rpy="0 0 0" />
-      <geometry>
-        <mesh filename="package://hdz_simplified/meshes/hdz_up_board_link.STL" />
-      </geometry>
-      <material name="">
-        <color rgba="0.5 0.5 0.6 1" />
-      </material>
-    </visual>
-    <collision>
-      <origin xyz="0 0 0" rpy="0 0 0" />
-      <geometry>
-        <mesh filename="package://hdz_simplified/meshes/hdz_up_board_link.STL" />
-      </geometry>
-    </collision>
-  </link>
-  <link name="hdz_steel_frame_link">
-    <inertial>
-      <origin xyz="0.0088033 8.2139E-17 0.14288" rpy="0 0 0" />
-      <mass value="15.553" />
-      <inertia ixx="0.42803" ixy="6.1895E-17" ixz="-0.037958"
-        iyy="0.31512" iyz="-1.7925E-17" izz="0.36" />
-    </inertial>
-    <visual>
-      <origin xyz="0 0 0" rpy="0 0 0" />
-      <geometry>
-        <mesh filename="package://hdz_simplified/meshes/hdz_steel_frame_link.STL" />
-      </geometry>
-      <material name="">
-        <color rgba="0.5 0.5 0.6 1" />
-      </material>
-    </visual>
-    <collision>
-      <origin xyz="0 0 0" rpy="0 0 0" />
-      <geometry>
-        <mesh filename="package://hdz_simplified/meshes/hdz_steel_frame_link.STL" />
-      </geometry>
-    </collision>
-  </link>
-  <joint name="hdz_base_joint" type="fixed">
-    <parent link="hdz_base_link" />
-    <child link="hdz_up_board_link" />
-    <origin xyz="0.0 0.0 0.482" rpy="0.0 0.0 0.0" />
-  </joint>
-  <joint name="hdz_steel_frame_joint" type="fixed">
-    <origin xyz="-0.23005 0 0.005" rpy="0 0 0" />
-    <parent link="hdz_up_board_link" />
-    <child link="hdz_steel_frame_link" />
-  </joint>
-  <joint name="hdz_arm_base_joint" type="fixed">
-    <origin xyz="0.203 0 0" rpy="0 0 0" />
-    <parent link="hdz_up_board_link" />
-    <child link="hdz_arm_base_link" />
+<robot xmlns:xacro="http://www.ros.org/wiki/xacro" name="hdz">
+  <link
+    name="hdz_base_link">
+    <inertial>
+      <origin
+        xyz="0.12543 -0.00028125 0.20317"
+        rpy="0 0 0" />
+      <mass
+        value="104.27" />
+      <inertia
+        ixx="1.0396"
+        ixy="-0.00012968"
+        ixz="-0.16582"
+        iyy="5.1965"
+        iyz="6.1158E-06"
+        izz="5.1293" />
+    </inertial>
+    <visual>
+      <origin
+        xyz="0 0 0"
+        rpy="0 0 0" />
+      <geometry>
+        <mesh
+          filename="package://hdz_simplified/meshes/hdz_base_link.STL" />
+      </geometry>
+      <material
+        name="">
+        <color
+          rgba="0.8 0.8 0.8 1" />
+      </material>
+    </visual>
+    <collision>
+      <origin
+        xyz="0 0 0"
+        rpy="0 0 0" />
+      <geometry>
+        <mesh
+          filename="package://hdz_simplified/meshes/hdz_base_link.STL" />
+      </geometry>
+    </collision>
+  </link>
+  <link
+    name="hdz_extend_board_link">
+    <inertial>
+      <origin
+        xyz="-0.066986 -5.6066E-15 0.0025"
+        rpy="0 0 0" />
+      <mass
+        value="5.8885" />
+      <inertia
+        ixx="0.25499"
+        ixy="4.1319E-16"
+        ixz="1.5274E-19"
+        iyy="0.0505"
+        iyz="9.9326E-16"
+        izz="0.30546" />
+    </inertial>
+    <visual>
+      <origin
+        xyz="0 0 0"
+        rpy="0 0 0" />
+      <geometry>
+        <mesh
+          filename="package://hdz_simplified/meshes/hdz_extend_board_link.STL" />
+      </geometry>
+      <material
+        name="">
+        <color
+          rgba="0.3 0.5 0.3 1" />
+      </material>
+    </visual>
+    <collision>
+      <origin
+        xyz="0 0 0"
+        rpy="0 0 0" />
+      <geometry>
+        <mesh
+          filename="package://hdz_simplified/meshes/hdz_extend_board_link.STL" />
+      </geometry>
+    </collision>
+  </link>
+  <joint
+    name="hdz_extend_board_joint"
+    type="fixed">
+    <origin
+      xyz="0.23816 0 0.4357"
+      rpy="0 0 0" />
+    <parent
+      link="hdz_base_link" />
+    <child
+      link="hdz_extend_board_link" />
+    <axis
+      xyz="0 0 0" />
+  </joint>
+  <link name="hdz_ur_base_link" />
+  <joint
+    name="hdz_ur_base_joint"
+    type="fixed">
+    <origin
+      xyz="0.13075 0 -0.09"
+      rpy="0 0 0" />
+    <parent
+      link="hdz_extend_board_link" />
+    <child
+      link="hdz_ur_base_link" />
+    <axis
+      xyz="0 0 0" />
+  </joint>
+  <link
+    name="hdz_steel_frame_link">
+    <inertial>
+      <origin
+        xyz="-0.1116 -0.020422 0.25051"
+        rpy="0 0 0" />
+      <mass
+        value="10.158" />
+      <inertia
+        ixx="0.09884"
+        ixy="5.6177E-06"
+        ixz="-3.3121E-07"
+        iyy="0.085565"
+        iyz="-8.766E-06"
+        izz="0.037015" />
+    </inertial>
+    <visual>
+      <origin
+        xyz="0 0 0"
+        rpy="0 0 0" />
+      <geometry>
+        <mesh
+          filename="package://hdz_simplified/meshes/hdz_steel_frame_link.STL" />
+      </geometry>
+      <material
+        name="">
+        <color
+          rgba="0.2 0.2 0.2 1" />
+      </material>
+    </visual>
+    <collision>
+      <origin
+        xyz="0 0 0"
+        rpy="0 0 0" />
+      <geometry>
+        <mesh
+          filename="package://hdz_simplified/meshes/hdz_steel_frame_link.STL" />
+      </geometry>
+    </collision>
+  </link>
+  <joint
+    name="hdz_steel_frame_joint"
+    type="fixed">
+    <origin
+      xyz="-0.29675 0 0.005"
+      rpy="0 0 0" />
+    <parent
+      link="hdz_extend_board_link" />
+    <child
+      link="hdz_steel_frame_link" />
+    <axis
+      xyz="0 0 0" />
+    <limit
+      lower="0"
+      upper="0"
+      effort="0"
+      velocity="0" />
+  </joint>
+  <link
+    name="hdz_ur_control_cabinet_link">
+    <inertial>
+      <origin
+        xyz="-0.00042578 4.3304E-05 0.052484"
+        rpy="0 0 0" />
+      <mass
+        value="0.96366" />
+      <inertia
+        ixx="0.016929"
+        ixy="-5.3803E-06"
+        ixz="1.9944E-06"
+        iyy="0.0096351"
+        iyz="3.1423E-06"
+        izz="0.022879" />
+    </inertial>
+    <visual>
+      <origin
+        xyz="0 0 0"
+        rpy="0 0 0" />
+      <geometry>
+        <mesh
+          filename="package://hdz_simplified/meshes/hdz_ur_control_cabinet_link.STL" />
+      </geometry>
+      <material
+        name="">
+        <color
+          rgba="0.2 0.2 0.2 1" />
+      </material>
+    </visual>
+    <collision>
+      <origin
+        xyz="0 0 0"
+        rpy="0 0 0" />
+      <geometry>
+        <mesh
+          filename="package://hdz_simplified/meshes/hdz_ur_control_cabinet_link.STL" />
+      </geometry>
+    </collision>
+  </link>
+  <joint
+    name="hdz_ur_control_cabinet_joint"
+    type="fixed">
+    <origin
+      xyz="0.0335 0 -0.005"
+      rpy="0 0 0" />
+    <parent
+      link="hdz_steel_frame_link" />
+    <child
+      link="hdz_ur_control_cabinet_link" />
+    <axis
+      xyz="0 0 0" />
   </joint>
 </robot>

File: ur_perception_description/urdf/ue5e_perception.urdf.xacro (robot description, xacro)
@@ -11,5 +11,5 @@
     </joint>
     <!-- UR model -->
-    <xacro:arg name="ur_parent" default="hdz_arm_base_link" />
+    <xacro:arg name="ur_parent" default="hdz_ur_base_link" />
     <xacro:include filename="$(find ur_perception_description)/urdf/ur5e.urdf.xacro" />
     <!-- RobotIQ Gripper -->

Commit message: tried to load mesh in gazebo but failed

File: hdz_simplified/urdf/hdz_simplified.xacro (robot description, xacro)
@@ -22,7 +22,10 @@
         rpy="0 0 0" />
       <geometry>
+        <box size="0.8 0.8 0.4" />
+      </geometry>
+      <!-- <geometry>
         <mesh
           filename="package://hdz_simplified/meshes/hdz_base_link.STL" />
-      </geometry>
+      </geometry> -->
       <material
         name="">
@@ -31,5 +34,5 @@
       </material>
     </visual>
-    <collision>
+    <!-- <collision>
       <origin
         xyz="0 0 0"
@@ -39,5 +42,5 @@
           filename="package://hdz_simplified/meshes/hdz_base_link.STL" />
       </geometry>
-    </collision>
+    </collision> -->
   </link>
   <link
@@ -62,7 +65,10 @@
         rpy="0 0 0" />
       <geometry>
+        <box size="0.2 0.2 0.2" />
+      </geometry>
+      <!-- <geometry>
         <mesh
           filename="package://hdz_simplified/meshes/hdz_extend_board_link.STL" />
-      </geometry>
+      </geometry> -->
       <material
         name="">
@@ -71,5 +77,5 @@
       </material>
     </visual>
-    <collision>
+    <!-- <collision>
       <origin
         xyz="0 0 0"
@@ -79,5 +85,5 @@
           filename="package://hdz_simplified/meshes/hdz_extend_board_link.STL" />
       </geometry>
-    </collision>
+    </collision> -->
   </link>
   <joint
@@ -128,23 +134,26 @@
         xyz="0 0 0"
         rpy="0 0 0" />
+      <!-- <geometry>
+        <box size="0.2 0.2 0.2" />
+      </geometry> -->
+      <geometry>
+        <mesh
+          filename="package://hdz_simplified/meshes/hdz_steel_frame_link.obj" />
+      </geometry>
+      <material
+        name="">
+        <color
+          rgba="0.2 0.2 0.2 1" />
+      </material>
+    </visual>
+    <!-- <collision>
+      <origin
+        xyz="0 0 0"
+        rpy="0 0 0" />
       <geometry>
         <mesh
           filename="package://hdz_simplified/meshes/hdz_steel_frame_link.STL" />
       </geometry>
-      <material
-        name="">
-        <color
-          rgba="0.2 0.2 0.2 1" />
-      </material>
-    </visual>
-    <collision>
-      <origin
-        xyz="0 0 0"
-        rpy="0 0 0" />
-      <geometry>
-        <mesh
-          filename="package://hdz_simplified/meshes/hdz_steel_frame_link.STL" />
-      </geometry>
-    </collision>
+    </collision> -->
   </link>
   <joint
@@ -187,7 +196,10 @@
         rpy="0 0 0" />
       <geometry>
+        <box size="0.2 0.2 0.2" />
+      </geometry>
+      <!-- <geometry>
         <mesh
           filename="package://hdz_simplified/meshes/hdz_ur_control_cabinet_link.STL" />
-      </geometry>
+      </geometry> -->
       <material
         name="">
@@ -196,5 +208,5 @@
       </material>
     </visual>
-    <collision>
+    <!-- <collision>
       <origin
         xyz="0 0 0"
@@ -204,5 +216,5 @@
           filename="package://hdz_simplified/meshes/hdz_ur_control_cabinet_link.STL" />
       </geometry>
-    </collision>
+    </collision> -->
   </link>
   <joint

File: ur_perception_description/urdf/ue5e_perception.urdf.xacro (robot description, xacro)
@@ -3,85 +3,34 @@
     <!-- create link fixed to the "world" -->
     <link name="world" />
+    <link name="robot_base" />
+    <joint name="robot_base_joint" type="fixed">
+        <parent link="world" />
+        <child link="robot_base" />
+        <origin xyz="0.0 1.0 1.0" rpy="0.0 0.0 0.0" />
+    </joint>
     <!-- 撼地者 -->
     <xacro:include filename="$(find hdz_simplified)/urdf/hdz_simplified.xacro" />
     <joint name="hdz_joint" type="fixed">
-        <parent link="world" />
+        <parent link="robot_base" />
         <child link="hdz_base_link" />
         <origin xyz="0.0 0.0 0.0" rpy="0.0 0.0 0.0" />
     </joint>
     <!-- UR model -->
-    <xacro:arg name="ur_parent" default="hdz_ur_base_link" />
-    <xacro:include filename="$(find ur_perception_description)/urdf/ur5e.urdf.xacro" />
-    <!-- RobotIQ Gripper -->
-    <xacro:include filename="$(find robotiq_description)/urdf/robotiq_2f_85_macro.urdf.xacro" />
-    <xacro:robotiq_gripper name="RobotiqGripperHardwareInterface" prefix="" parent="tool0"
-        use_fake_hardware="true">
-        <origin xyz="0 0 0" rpy="0 0 0" />
-    </xacro:robotiq_gripper>
-    <ros2_control name="RobotIQGazeboSystem" type="system">
-        <hardware>
-            <plugin>gazebo_ros2_control/GazeboSystem</plugin>
-        </hardware>
-        <joint name="robotiq_85_left_knuckle_joint">
-            <command_interface name="position" />
-            <state_interface name="position" />
-            <state_interface name="velocity" />
-            <state_interface name="effort" />
-        </joint>
-        <joint name="robotiq_85_right_knuckle_joint">
-            <!-- <param name="mimic">robotiq_85_left_knuckle_joint</param>
-            <param name="multiplier">-1</param> -->
-            <command_interface name="position" />
-            <state_interface name="position" />
-            <state_interface name="velocity" />
-            <state_interface name="effort" />
-        </joint>
-        <joint name="robotiq_85_left_inner_knuckle_joint">
-            <!-- <param name="mimic">robotiq_85_left_knuckle_joint</param>
-            <param name="multiplier">1</param> -->
-            <command_interface name="position" />
-            <state_interface name="position" />
-            <state_interface name="velocity" />
-            <state_interface name="effort" />
-        </joint>
-        <joint name="robotiq_85_right_inner_knuckle_joint">
-            <!-- <param name="mimic">robotiq_85_left_knuckle_joint</param>
-            <param name="multiplier">-1</param> -->
-            <command_interface name="position" />
-            <state_interface name="position" />
-            <state_interface name="velocity" />
-            <state_interface name="effort" />
-        </joint>
-        <joint name="robotiq_85_left_finger_tip_joint">
-            <!-- <param name="mimic">robotiq_85_left_knuckle_joint</param>
-            <param name="multiplier">-1</param> -->
-            <command_interface name="position" />
-            <state_interface name="position" />
-            <state_interface name="velocity" />
-            <state_interface name="effort" />
-        </joint>
-        <joint name="robotiq_85_right_finger_tip_joint">
-            <!-- <param name="mimic">robotiq_85_left_knuckle_joint</param>
-            <param name="multiplier">1</param> -->
-            <command_interface name="position" />
-            <state_interface name="position" />
-            <state_interface name="velocity" />
-            <state_interface name="effort" />
-        </joint>
-    </ros2_control>
+    <!-- <xacro:arg name="ur_parent" default="hdz_ur_base_link" />
+    <xacro:include filename="$(find ur_perception_description)/urdf/ur5e.urdf.xacro" /> -->
     <!-- d435i model -->
-    <xacro:arg name="use_nominal_extrinsics" default="false" />
+    <!-- <xacro:arg name="use_nominal_extrinsics" default="false" />
     <xacro:include filename="$(find realsense2_description)/urdf/_d435i.urdf.xacro" />
     <xacro:sensor_d435i parent="base"
         use_nominal_extrinsics="$(arg use_nominal_extrinsics)">
         <origin xyz="0.0 0.0 2" rpy="0.0 ${pi/2} 0.0" />
-    </xacro:sensor_d435i>
+    </xacro:sensor_d435i> -->
     <!-- gazebo camera -->
-    <joint name="camera_optical_joint" type="fixed">
+    <!-- <joint name="camera_optical_joint" type="fixed">
         <origin xyz="0 0 0" rpy="${-pi/2} 0 ${-pi/2}" />
         <parent link="camera_link" />
         <child link="camera_link_optical" />
-    </joint>
-    <link name="camera_link_optical"></link>
+    </joint> -->
+    <!-- <link name="camera_link_optical"></link> -->
     <!-- Add a gazebo tag for the ORIGINAL camera_link (but in the plugin we reference the optical
     frame so that ROS can orient things correctly) -->
@@ -91,5 +40,5 @@
     <!-- Note that although visualise is set to true, it won't actually visualise the depth camera
     in gazebo. To see the preview, try swapping "depth" to "camera"-->
-    <gazebo reference="camera_link">
+    <!-- <gazebo reference="camera_link">
         <sensor type="depth" name="my_camera">
             <update_rate>20</update_rate>
@@ -118,4 +67,4 @@
             </plugin>
         </sensor>
-    </gazebo>
+    </gazebo> -->
 </robot>

Commit message: 新模型完成！！！

File: hdz_simplified/urdf/hdz_simplified.xacro (robot description, xacro)
@@ -22,10 +22,6 @@
         rpy="0 0 0" />
       <geometry>
-        <box size="0.8 0.8 0.4" />
-      </geometry>
-      <!-- <geometry>
-        <mesh
-          filename="package://hdz_simplified/meshes/hdz_base_link.STL" />
-      </geometry> -->
+        <mesh filename="file://$(find hdz_simplified)/meshes/hdz_base_link.STL" />
+      </geometry>
       <material
         name="">
@@ -40,5 +36,5 @@
       <geometry>
         <mesh
-          filename="package://hdz_simplified/meshes/hdz_base_link.STL" />
+          filename="file://$(find hdz_simplified)/meshes/hdz_base_link.STL" />
       </geometry>
     </collision> -->
@@ -65,10 +61,7 @@
         rpy="0 0 0" />
       <geometry>
-        <box size="0.2 0.2 0.2" />
-      </geometry>
-      <!-- <geometry>
-        <mesh
-          filename="package://hdz_simplified/meshes/hdz_extend_board_link.STL" />
-      </geometry> -->
+        <mesh
+          filename="file://$(find hdz_simplified)/meshes/hdz_extend_board_link.STL" />
+      </geometry>
       <material
         name="">
@@ -77,13 +70,13 @@
       </material>
     </visual>
-    <!-- <collision>
-      <origin
-        xyz="0 0 0"
-        rpy="0 0 0" />
-      <geometry>
-        <mesh
-          filename="package://hdz_simplified/meshes/hdz_extend_board_link.STL" />
-      </geometry>
-    </collision> -->
+    <collision>
+      <origin
+        xyz="0 0 0"
+        rpy="0 0 0" />
+      <geometry>
+        <mesh
+          filename="file://$(find hdz_simplified)/meshes/hdz_extend_board_link.STL" />
+      </geometry>
+    </collision>
   </link>
   <joint
@@ -134,10 +127,7 @@
         xyz="0 0 0"
         rpy="0 0 0" />
-      <!-- <geometry>
-        <box size="0.2 0.2 0.2" />
-      </geometry> -->
-      <geometry>
-        <mesh
-          filename="package://hdz_simplified/meshes/hdz_steel_frame_link.obj" />
+      <geometry>
+        <mesh
+          filename="file://$(find hdz_simplified)/meshes/hdz_steel_frame_link.STL" />
       </geometry>
       <material
@@ -147,13 +137,12 @@
       </material>
     </visual>
-    <!-- <collision>
-      <origin
-        xyz="0 0 0"
-        rpy="0 0 0" />
-      <geometry>
-        <mesh
-          filename="package://hdz_simplified/meshes/hdz_steel_frame_link.STL" />
-      </geometry>
-    </collision> -->
+    <collision>
+      <origin
+        xyz="0 0 0"
+        rpy="0 0 0" />
+      <geometry>
+        <mesh filename="file://$(find hdz_simplified)/meshes/hdz_steel_frame_link.STL" />
+      </geometry>
+    </collision>
   </link>
   <joint
@@ -196,10 +185,7 @@
         rpy="0 0 0" />
       <geometry>
-        <box size="0.2 0.2 0.2" />
-      </geometry>
-      <!-- <geometry>
-        <mesh
-          filename="package://hdz_simplified/meshes/hdz_ur_control_cabinet_link.STL" />
-      </geometry> -->
+        <mesh
+          filename="file://$(find hdz_simplified)/meshes/hdz_ur_control_cabinet_link.STL" />
+      </geometry>
       <material
         name="">
@@ -208,13 +194,13 @@
       </material>
     </visual>
-    <!-- <collision>
-      <origin
-        xyz="0 0 0"
-        rpy="0 0 0" />
-      <geometry>
-        <mesh
-          filename="package://hdz_simplified/meshes/hdz_ur_control_cabinet_link.STL" />
-      </geometry>
-    </collision> -->
+    <collision>
+      <origin
+        xyz="0 0 0"
+        rpy="0 0 0" />
+      <geometry>
+        <mesh
+          filename="file://$(find hdz_simplified)/meshes/hdz_ur_control_cabinet_link.STL" />
+      </geometry>
+    </collision>
   </link>
   <joint

File: ur_perception_description/urdf/ue5e_perception.urdf.xacro (robot description, xacro)
@@ -7,5 +7,5 @@
         <parent link="world" />
         <child link="robot_base" />
-        <origin xyz="0.0 1.0 1.0" rpy="0.0 0.0 0.0" />
+        <origin xyz="0.0 0.0 0.0" rpy="0.0 0.0 0.0" />
     </joint>
     <!-- 撼地者 -->
@@ -17,20 +17,20 @@
     </joint>
     <!-- UR model -->
-    <!-- <xacro:arg name="ur_parent" default="hdz_ur_base_link" />
-    <xacro:include filename="$(find ur_perception_description)/urdf/ur5e.urdf.xacro" /> -->
+    <xacro:arg name="ur_parent" default="hdz_ur_base_link" />
+    <xacro:include filename="$(find ur_perception_description)/urdf/ur5e.urdf.xacro" />
     <!-- d435i model -->
-    <!-- <xacro:arg name="use_nominal_extrinsics" default="false" />
+    <xacro:arg name="use_nominal_extrinsics" default="false" />
     <xacro:include filename="$(find realsense2_description)/urdf/_d435i.urdf.xacro" />
     <xacro:sensor_d435i parent="base"
         use_nominal_extrinsics="$(arg use_nominal_extrinsics)">
         <origin xyz="0.0 0.0 2" rpy="0.0 ${pi/2} 0.0" />
-    </xacro:sensor_d435i> -->
+    </xacro:sensor_d435i>
     <!-- gazebo camera -->
-    <!-- <joint name="camera_optical_joint" type="fixed">
+    <joint name="camera_optical_joint" type="fixed">
         <origin xyz="0 0 0" rpy="${-pi/2} 0 ${-pi/2}" />
         <parent link="camera_link" />
         <child link="camera_link_optical" />
-    </joint> -->
-    <!-- <link name="camera_link_optical"></link> -->
+    </joint>
+    <link name="camera_link_optical"></link>
     <!-- Add a gazebo tag for the ORIGINAL camera_link (but in the plugin we reference the optical
     frame so that ROS can orient things correctly) -->
@@ -40,5 +40,5 @@
     <!-- Note that although visualise is set to true, it won't actually visualise the depth camera
     in gazebo. To see the preview, try swapping "depth" to "camera"-->
-    <!-- <gazebo reference="camera_link">
+    <gazebo reference="camera_link">
         <sensor type="depth" name="my_camera">
             <update_rate>20</update_rate>
@@ -67,4 +67,4 @@
             </plugin>
         </sensor>
-    </gazebo> -->
+    </gazebo>
 </robot>
