Commit message: 新模型完成！！！

File: ur_perception_moveit_launcher/srdf/ur_macro.srdf.xacro (robot description, xacro)
@@ -1,18 +1,33 @@
 <?xml version="1.0" encoding="UTF-8"?>
 <robot xmlns:xacro="http://wiki.ros.org/xacro">
-<!--This does not replace URDF, and is not an extension of URDF.
+  <!--This
+  does not replace URDF, and is not an extension of URDF.
     This is a format for representing semantic information about the robot structure.
-    A URDF file must exist for this robot as well, where the joints and the links that are referenced are defined
+    A URDF file must exist for this robot as well, where the joints and the links that are referenced
+  are defined
 -->
   <xacro:macro name="ur_srdf" params="name prefix">
-    <!--GROUPS - Representation of a set of joints and links. This can be useful for specifying DOF to plan for, defining arms, end effectors, etc-->
-    <!--LINKS - When a link is specified, the parent joint of that link (if it exists) is automatically included-->
-    <!--JOINTS - When a joint is specified, the child link of that joint (which will always exist) is automatically included-->
-    <!--CHAINS - When a chain is specified, all the links along the chain (including endpoints) are included in the group. Additionally, all the joints that are parents to included links are also included. This means that joints along the chain and the parent joint of the base link are included in the group-->
-    <!--SUBGROUPS - Groups can also be formed by referencing to already defined group names-->
+    <!--GROUPS
+    - Representation of a set of joints and links. This can be useful for specifying DOF to plan
+    for, defining arms, end effectors, etc-->
+    <!--LINKS
+    - When a link is specified, the parent joint of that link (if it exists) is automatically
+    included-->
+    <!--JOINTS
+    - When a joint is specified, the child link of that joint (which will always exist) is
+    automatically included-->
+    <!--CHAINS
+    - When a chain is specified, all the links along the chain (including endpoints) are included in
+    the group. Additionally, all the joints that are parents to included links are also included.
+    This means that joints along the chain and the parent joint of the base link are included in the
+    group-->
+    <!--SUBGROUPS
+    - Groups can also be formed by referencing to already defined group names-->
     <group name="${prefix}${name}_manipulator">
       <chain base_link="${prefix}base_link" tip_link="${prefix}tool0" />
     </group>
-    <!--GROUP STATES - Purpose - Define a named state for a particular group, in terms of joint values. This is useful to define states like 'folded arms'-->
+    <!--GROUP
+    STATES - Purpose - Define a named state for a particular group, in terms of joint values. This
+    is useful to define states like 'folded arms'-->
     <group_state name="${prefix}home" group="${prefix}${name}_manipulator">
       <joint name="${prefix}elbow_joint" value="0" />
@@ -31,109 +46,50 @@
       <joint name="${prefix}wrist_3_joint" value="0" />
     </group_state>
-    <group_state name="${prefix}test_configuration" group="${prefix}${name}_manipulator">
-      <joint name="${prefix}elbow_joint" value="1.4" />
-      <joint name="${prefix}shoulder_lift_joint" value="-1.62" />
-      <joint name="${prefix}shoulder_pan_joint" value="1.54" />
-      <joint name="${prefix}wrist_1_joint" value="-1.2" />
-      <joint name="${prefix}wrist_2_joint" value="-1.6" />
-      <joint name="${prefix}wrist_3_joint" value="-0.11" />
+    <group_state name="fold" group="${prefix}${name}_manipulator">
+      <joint name="elbow_joint" value="2.7317" />
+      <joint name="shoulder_lift_joint" value="-2.6635" />
+      <joint name="shoulder_pan_joint" value="0.2049" />
+      <joint name="wrist_1_joint" value="-3.14" />
+      <joint name="wrist_2_joint" value="-1.57" />
+      <joint name="wrist_3_joint" value="0" />
     </group_state>
-    <!--END EFFECTOR - Purpose - Represent information about an end effector.-->
-    <!--VIRTUAL JOINT - Purpose - this element defines a virtual joint between a robot link and an external frame of reference (considered fixed with respect to the robot)-->
-    <!--DISABLE COLLISIONS - By default it is assumed that any link of the robot could potentially come into collision with any other link in the robot. This tag disables collision checking between a specified pair of links. -->
-    <disable_collisions link1="base_link_inertia" link2="camera_link" reason="Adjacent"/>
-    <disable_collisions link1="base_link_inertia" link2="hdz_arm_frame" reason="Never"/>
-    <disable_collisions link1="base_link_inertia" link2="hdz_up_board" reason="Adjacent"/>
-    <disable_collisions link1="base_link_inertia" link2="shoulder_link" reason="Adjacent"/>
-    <disable_collisions link1="camera_link" link2="forearm_link" reason="Never"/>
-    <disable_collisions link1="camera_link" link2="hdz_arm_frame" reason="Never"/>
-    <disable_collisions link1="camera_link" link2="hdz_up_board" reason="Adjacent"/>
-    <disable_collisions link1="camera_link" link2="robotiq_85_base_link" reason="Never"/>
-    <disable_collisions link1="camera_link" link2="robotiq_85_left_finger_link" reason="Never"/>
-    <disable_collisions link1="camera_link" link2="robotiq_85_left_finger_tip_link" reason="Never"/>
-    <disable_collisions link1="camera_link" link2="robotiq_85_left_inner_knuckle_link" reason="Never"/>
-    <disable_collisions link1="camera_link" link2="robotiq_85_left_knuckle_link" reason="Never"/>
-    <disable_collisions link1="camera_link" link2="robotiq_85_right_finger_link" reason="Never"/>
-    <disable_collisions link1="camera_link" link2="robotiq_85_right_finger_tip_link" reason="Never"/>
-    <disable_collisions link1="camera_link" link2="robotiq_85_right_inner_knuckle_link" reason="Never"/>
-    <disable_collisions link1="camera_link" link2="robotiq_85_right_knuckle_link" reason="Never"/>
-    <disable_collisions link1="camera_link" link2="shoulder_link" reason="Never"/>
-    <disable_collisions link1="camera_link" link2="upper_arm_link" reason="Never"/>
-    <disable_collisions link1="camera_link" link2="wrist_1_link" reason="Never"/>
-    <disable_collisions link1="camera_link" link2="wrist_2_link" reason="Never"/>
-    <disable_collisions link1="camera_link" link2="wrist_3_link" reason="Never"/>
-    <disable_collisions link1="forearm_link" link2="upper_arm_link" reason="Adjacent"/>
-    <disable_collisions link1="forearm_link" link2="wrist_1_link" reason="Adjacent"/>
-    <disable_collisions link1="forearm_link" link2="wrist_2_link" reason="Never"/>
-    <disable_collisions link1="hdz_arm_frame" link2="hdz_up_board" reason="Adjacent"/>
-    <disable_collisions link1="hdz_arm_frame" link2="shoulder_link" reason="Never"/>
-    <disable_collisions link1="hdz_up_board" link2="shoulder_link" reason="Never"/>
-    <disable_collisions link1="robotiq_85_base_link" link2="robotiq_85_left_finger_link" reason="Never"/>
-    <disable_collisions link1="robotiq_85_base_link" link2="robotiq_85_left_finger_tip_link" reason="Never"/>
-    <disable_collisions link1="robotiq_85_base_link" link2="robotiq_85_left_inner_knuckle_link" reason="Adjacent"/>
-    <disable_collisions link1="robotiq_85_base_link" link2="robotiq_85_left_knuckle_link" reason="Adjacent"/>
-    <disable_collisions link1="robotiq_85_base_link" link2="robotiq_85_right_finger_link" reason="Never"/>
-    <disable_collisions link1="robotiq_85_base_link" link2="robotiq_85_right_finger_tip_link" reason="Never"/>
-    <disable_collisions link1="robotiq_85_base_link" link2="robotiq_85_right_inner_knuckle_link" reason="Adjacent"/>
-    <disable_collisions link1="robotiq_85_base_link" link2="robotiq_85_right_knuckle_link" reason="Adjacent"/>
-    <disable_collisions link1="robotiq_85_base_link" link2="wrist_1_link" reason="Never"/>
-    <disable_collisions link1="robotiq_85_base_link" link2="wrist_2_link" reason="Never"/>
-    <disable_collisions link1="robotiq_85_base_link" link2="wrist_3_link" reason="Adjacent"/>
-    <disable_collisions link1="robotiq_85_left_finger_link" link2="robotiq_85_left_finger_tip_link" reason="Adjacent"/>
-    <disable_collisions link1="robotiq_85_left_finger_link" link2="robotiq_85_left_inner_knuckle_link" reason="Never"/>
-    <disable_collisions link1="robotiq_85_left_finger_link" link2="robotiq_85_left_knuckle_link" reason="Adjacent"/>
-    <disable_collisions link1="robotiq_85_left_finger_link" link2="robotiq_85_right_finger_link" reason="Never"/>
-    <disable_collisions link1="robotiq_85_left_finger_link" link2="robotiq_85_right_finger_tip_link" reason="Never"/>
-    <disable_collisions link1="robotiq_85_left_finger_link" link2="robotiq_85_right_inner_knuckle_link" reason="Never"/>
-    <disable_collisions link1="robotiq_85_left_finger_link" link2="robotiq_85_right_knuckle_link" reason="Never"/>
-    <disable_collisions link1="robotiq_85_left_finger_link" link2="wrist_1_link" reason="Never"/>
-    <disable_collisions link1="robotiq_85_left_finger_link" link2="wrist_2_link" reason="Never"/>
-    <disable_collisions link1="robotiq_85_left_finger_link" link2="wrist_3_link" reason="Never"/>
-    <disable_collisions link1="robotiq_85_left_finger_tip_link" link2="robotiq_85_left_inner_knuckle_link" reason="Default"/>
-    <disable_collisions link1="robotiq_85_left_finger_tip_link" link2="robotiq_85_left_knuckle_link" reason="Never"/>
-    <disable_collisions link1="robotiq_85_left_finger_tip_link" link2="robotiq_85_right_finger_link" reason="Never"/>
-    <disable_collisions link1="robotiq_85_left_finger_tip_link" link2="robotiq_85_right_finger_tip_link" reason="Never"/>
-    <disable_collisions link1="robotiq_85_left_finger_tip_link" link2="robotiq_85_right_inner_knuckle_link" reason="Never"/>
-    <disable_collisions link1="robotiq_85_left_finger_tip_link" link2="robotiq_85_right_knuckle_link" reason="Never"/>
-    <disable_collisions link1="robotiq_85_left_finger_tip_link" link2="wrist_1_link" reason="Never"/>
-    <disable_collisions link1="robotiq_85_left_finger_tip_link" link2="wrist_2_link" reason="Never"/>
-    <disable_collisions link1="robotiq_85_left_finger_tip_link" link2="wrist_3_link" reason="Never"/>
-    <disable_collisions link1="robotiq_85_left_inner_knuckle_link" link2="robotiq_85_left_knuckle_link" reason="Never"/>
-    <disable_collisions link1="robotiq_85_left_inner_knuckle_link" link2="robotiq_85_right_finger_link" reason="Never"/>
-    <disable_collisions link1="robotiq_85_left_inner_knuckle_link" link2="robotiq_85_right_finger_tip_link" reason="Never"/>
-    <disable_collisions link1="robotiq_85_left_inner_knuckle_link" link2="robotiq_85_right_inner_knuckle_link" reason="Never"/>
-    <disable_collisions link1="robotiq_85_left_inner_knuckle_link" link2="robotiq_85_right_knuckle_link" reason="Never"/>
-    <disable_collisions link1="robotiq_85_left_inner_knuckle_link" link2="wrist_1_link" reason="Never"/>
-    <disable_collisions link1="robotiq_85_left_inner_knuckle_link" link2="wrist_2_link" reason="Never"/>
-    <disable_collisions link1="robotiq_85_left_inner_knuckle_link" link2="wrist_3_link" reason="Never"/>
-    <disable_collisions link1="robotiq_85_left_knuckle_link" link2="robotiq_85_right_finger_link" reason="Never"/>
-    <disable_collisions link1="robotiq_85_left_knuckle_link" link2="robotiq_85_right_finger_tip_link" reason="Never"/>
-    <disable_collisions link1="robotiq_85_left_knuckle_link" link2="robotiq_85_right_inner_knuckle_link" reason="Never"/>
-    <disable_collisions link1="robotiq_85_left_knuckle_link" link2="robotiq_85_right_knuckle_link" reason="Never"/>
-    <disable_collisions link1="robotiq_85_left_knuckle_link" link2="wrist_1_link" reason="Never"/>
-    <disable_collisions link1="robotiq_85_left_knuckle_link" link2="wrist_2_link" reason="Never"/>
-    <disable_collisions link1="robotiq_85_left_knuckle_link" link2="wrist_3_link" reason="Never"/>
-    <disable_collisions link1="robotiq_85_right_finger_link" link2="robotiq_85_right_finger_tip_link" reason="Adjacent"/>
-    <disable_collisions link1="robotiq_85_right_finger_link" link2="robotiq_85_right_inner_knuckle_link" reason="Never"/>
-    <disable_collisions link1="robotiq_85_right_finger_link" link2="robotiq_85_right_knuckle_link" reason="Adjacent"/>
-    <disable_collisions link1="robotiq_85_right_finger_link" link2="wrist_1_link" reason="Never"/>
-    <disable_collisions link1="robotiq_85_right_finger_link" link2="wrist_2_link" reason="Never"/>
-    <disable_collisions link1="robotiq_85_right_finger_link" link2="wrist_3_link" reason="Never"/>
-    <disable_collisions link1="robotiq_85_right_finger_tip_link" link2="robotiq_85_right_inner_knuckle_link" reason="Default"/>
-    <disable_collisions link1="robotiq_85_right_finger_tip_link" link2="robotiq_85_right_knuckle_link" reason="Never"/>
-    <disable_collisions link1="robotiq_85_right_finger_tip_link" link2="wrist_1_link" reason="Never"/>
-    <disable_collisions link1="robotiq_85_right_finger_tip_link" link2="wrist_2_link" reason="Never"/>
-    <disable_collisions link1="robotiq_85_right_finger_tip_link" link2="wrist_3_link" reason="Never"/>
-    <disable_collisions link1="robotiq_85_right_inner_knuckle_link" link2="robotiq_85_right_knuckle_link" reason="Never"/>
-    <disable_collisions link1="robotiq_85_right_inner_knuckle_link" link2="wrist_1_link" reason="Never"/>
-    <disable_collisions link1="robotiq_85_right_inner_knuckle_link" link2="wrist_2_link" reason="Never"/>
-    <disable_collisions link1="robotiq_85_right_inner_knuckle_link" link2="wrist_3_link" reason="Never"/>
-    <disable_collisions link1="robotiq_85_right_knuckle_link" link2="wrist_1_link" reason="Never"/>
-    <disable_collisions link1="robotiq_85_right_knuckle_link" link2="wrist_2_link" reason="Never"/>
-    <disable_collisions link1="robotiq_85_right_knuckle_link" link2="wrist_3_link" reason="Never"/>
-    <disable_collisions link1="shoulder_link" link2="upper_arm_link" reason="Adjacent"/>
-    <disable_collisions link1="wrist_1_link" link2="wrist_2_link" reason="Adjacent"/>
-    <disable_collisions link1="wrist_1_link" link2="wrist_3_link" reason="Never"/>
-    <disable_collisions link1="wrist_2_link" link2="wrist_3_link" reason="Adjacent"/>
+    <!--END
+    EFFECTOR - Purpose - Represent information about an end effector.-->
+    <!--VIRTUAL
+    JOINT - Purpose - this element defines a virtual joint between a robot link and an external
+    frame of reference (considered fixed with respect to the robot)-->
+    <!--DISABLE
+    COLLISIONS - By default it is assumed that any link of the robot could potentially come into
+    collision with any other link in the robot. This tag disables collision checking between a
+    specified pair of links. -->
+    <disable_collisions link1="base_link_inertia" link2="camera_link" reason="Adjacent" />
+    <disable_collisions link1="base_link_inertia" link2="hdz_extend_board_link" reason="Adjacent" />
+    <disable_collisions link1="base_link_inertia" link2="hdz_steel_frame_link" reason="Never" />
+    <disable_collisions link1="base_link_inertia" link2="hdz_ur_control_cabinet_link" reason="Never" />
+    <disable_collisions link1="base_link_inertia" link2="shoulder_link" reason="Adjacent" />
+    <disable_collisions link1="camera_link" link2="forearm_link" reason="Never" />
+    <disable_collisions link1="camera_link" link2="hdz_extend_board_link" reason="Adjacent" />
+    <disable_collisions link1="camera_link" link2="hdz_steel_frame_link" reason="Never" />
+    <disable_collisions link1="camera_link" link2="hdz_ur_control_cabinet_link" reason="Never" />
+    <disable_collisions link1="camera_link" link2="shoulder_link" reason="Never" />
+    <disable_collisions link1="camera_link" link2="upper_arm_link" reason="Never" />
+    <disable_collisions link1="camera_link" link2="wrist_1_link" reason="Never" />
+    <disable_collisions link1="camera_link" link2="wrist_2_link" reason="Never" />
+    <disable_collisions link1="camera_link" link2="wrist_3_link" reason="Never" />
+    <disable_collisions link1="forearm_link" link2="upper_arm_link" reason="Adjacent" />
+    <disable_collisions link1="forearm_link" link2="wrist_1_link" reason="Adjacent" />
+    <disable_collisions link1="forearm_link" link2="wrist_2_link" reason="Never" />
+    <disable_collisions link1="hdz_extend_board_link" link2="hdz_steel_frame_link" reason="Adjacent" />
+    <disable_collisions link1="hdz_extend_board_link" link2="hdz_ur_control_cabinet_link"
+      reason="Default" />
+    <disable_collisions link1="hdz_extend_board_link" link2="shoulder_link" reason="Never" />
+    <disable_collisions link1="hdz_steel_frame_link" link2="hdz_ur_control_cabinet_link"
+      reason="Adjacent" />
+    <disable_collisions link1="hdz_steel_frame_link" link2="shoulder_link" reason="Never" />
+    <disable_collisions link1="hdz_ur_control_cabinet_link" link2="shoulder_link" reason="Never" />
+    <disable_collisions link1="shoulder_link" link2="upper_arm_link" reason="Adjacent" />
+    <disable_collisions link1="wrist_1_link" link2="wrist_2_link" reason="Adjacent" />
+    <disable_collisions link1="wrist_1_link" link2="wrist_3_link" reason="Never" />
+    <disable_collisions link1="wrist_2_link" link2="wrist_3_link" reason="Adjacent" />
   </xacro:macro>
 </robot>
