Commit message: cleanup many code

File: hdz_simplified/urdf/hdz_simplified.xacro (robot description, xacro)
@@ -1,219 +1,8 @@
 <?xml version="1.0" encoding="utf-8"?>
 <robot xmlns:xacro="http://www.ros.org/wiki/xacro" name="hdz">
-  <link
-    name="hdz_base_link">
-    <inertial>
-      <origin
-        xyz="0.12543 -0.00028125 0.20317"
-        rpy="0 0 0" />
-      <mass
-        value="104.27" />
-      <inertia
-        ixx="1.0396"
-        ixy="-0.00012968"
-        ixz="-0.16582"
-        iyy="5.1965"
-        iyz="6.1158E-06"
-        izz="5.1293" />
-    </inertial>
-    <visual>
-      <origin
-        xyz="0 0 0"
-        rpy="0 0 0" />
-      <geometry>
-        <mesh filename="file://$(find hdz_simplified)/meshes/hdz_base_link.STL" />
-      </geometry>
-      <material
-        name="">
-        <color
-          rgba="0.8 0.8 0.8 1" />
-      </material>
-    </visual>
-    <!-- <collision>
-      <origin
-        xyz="0 0 0"
-        rpy="0 0 0" />
-      <geometry>
-        <mesh
-          filename="file://$(find hdz_simplified)/meshes/hdz_base_link.STL" />
-      </geometry>
-    </collision> -->
-  </link>
-  <link
-    name="hdz_extend_board_link">
-    <inertial>
-      <origin
-        xyz="-0.066986 -5.6066E-15 0.0025"
-        rpy="0 0 0" />
-      <mass
-        value="5.8885" />
-      <inertia
-        ixx="0.25499"
-        ixy="4.1319E-16"
-        ixz="1.5274E-19"
-        iyy="0.0505"
-        iyz="9.9326E-16"
-        izz="0.30546" />
-    </inertial>
-    <visual>
-      <origin
-        xyz="0 0 0"
-        rpy="0 0 0" />
-      <geometry>
-        <mesh
-          filename="file://$(find hdz_simplified)/meshes/hdz_extend_board_link.STL" />
-      </geometry>
-      <material
-        name="">
-        <color
-          rgba="0.3 0.5 0.3 1" />
-      </material>
-    </visual>
-    <collision>
-      <origin
-        xyz="0 0 0"
-        rpy="0 0 0" />
-      <geometry>
-        <mesh
-          filename="file://$(find hdz_simplified)/meshes/hdz_extend_board_link.STL" />
-      </geometry>
-    </collision>
-  </link>
-  <joint
-    name="hdz_extend_board_joint"
-    type="fixed">
-    <origin
-      xyz="0.23816 0 0.4357"
-      rpy="0 0 0" />
-    <parent
-      link="hdz_base_link" />
-    <child
-      link="hdz_extend_board_link" />
-    <axis
-      xyz="0 0 0" />
-  </joint>
-  <link name="hdz_ur_base_link" />
-  <joint
-    name="hdz_ur_base_joint"
-    type="fixed">
-    <origin
-      xyz="0.13075 0 -0.09"
-      rpy="0 0 0" />
-    <parent
-      link="hdz_extend_board_link" />
-    <child
-      link="hdz_ur_base_link" />
-    <axis
-      xyz="0 0 0" />
-  </joint>
-  <link
-    name="hdz_steel_frame_link">
-    <inertial>
-      <origin
-        xyz="-0.1116 -0.020422 0.25051"
-        rpy="0 0 0" />
-      <mass
-        value="10.158" />
-      <inertia
-        ixx="0.09884"
-        ixy="5.6177E-06"
-        ixz="-3.3121E-07"
-        iyy="0.085565"
-        iyz="-8.766E-06"
-        izz="0.037015" />
-    </inertial>
-    <visual>
-      <origin
-        xyz="0 0 0"
-        rpy="0 0 0" />
-      <geometry>
-        <mesh
-          filename="file://$(find hdz_simplified)/meshes/hdz_steel_frame_link.STL" />
-      </geometry>
-      <material
-        name="">
-        <color
-          rgba="0.2 0.2 0.2 1" />
-      </material>
-    </visual>
-    <collision>
-      <origin
-        xyz="0 0 0"
-        rpy="0 0 0" />
-      <geometry>
-        <mesh filename="file://$(find hdz_simplified)/meshes/hdz_steel_frame_link.STL" />
-      </geometry>
-    </collision>
-  </link>
-  <joint
-    name="hdz_steel_frame_joint"
-    type="fixed">
-    <origin
-      xyz="-0.29675 0 0.005"
-      rpy="0 0 0" />
-    <parent
-      link="hdz_extend_board_link" />
-    <child
-      link="hdz_steel_frame_link" />
-    <axis
-      xyz="0 0 0" />
-    <limit
-      lower="0"
-      upper="0"
-      effort="0"
-      velocity="0" />
-  </joint>
-  <link
-    name="hdz_ur_control_cabinet_link">
-    <inertial>
-      <origin
-        xyz="-0.00042578 4.3304E-05 0.052484"
-        rpy="0 0 0" />
-      <mass
-        value="0.96366" />
-      <inertia
-        ixx="0.016929"
-        ixy="-5.3803E-06"
-        ixz="1.9944E-06"
-        iyy="0.0096351"
-        iyz="3.1423E-06"
-        izz="0.022879" />
-    </inertial>
-    <visual>
-      <origin
-        xyz="0 0 0"
-        rpy="0 0 0" />
-      <geometry>
-        <mesh
-          filename="file://$(find hdz_simplified)/meshes/hdz_ur_control_cabinet_link.STL" />
-      </geometry>
-      <material
-        name="">
-        <color
-          rgba="0.2 0.2 0.2 1" />
-      </material>
-    </visual>
-    <collision>
-      <origin
-        xyz="0 0 0"
-        rpy="0 0 0" />
-      <geometry>
-        <mesh
-          filename="file://$(find hdz_simplified)/meshes/hdz_ur_control_cabinet_link.STL" />
-      </geometry>
-    </collision>
-  </link>
-  <joint
-    name="hdz_ur_control_cabinet_joint"
-    type="fixed">
-    <origin
-      xyz="0.0335 0 -0.005"
-      rpy="0 0 0" />
-    <parent
-      link="hdz_steel_frame_link" />
-    <child
-      link="hdz_ur_control_cabinet_link" />
-    <axis
-      xyz="0 0 0" />
-  </joint>
+  <xacro:include filename="$(find hdz_simplified)/urdf/hdz_simplified_macro.xacro" />
+  <link name="world" />
+  <xacro:hdz_simplified parent="world" tf_prefix="hdz_">
+    <origin xyz="0 0 0" rpy="0 0 0" />
+  </xacro:hdz_simplified>
 </robot>

File: ur_perception_description/urdf/ue5e_perception.urdf.xacro (robot description, xacro)
@@ -3,68 +3,11 @@
     <!-- create link fixed to the "world" -->
     <link name="world" />
-    <link name="robot_base" />
-    <joint name="robot_base_joint" type="fixed">
-        <parent link="world" />
-        <child link="robot_base" />
-        <origin xyz="0.0 0.62 0.19" rpy="0.0 0.0 -1.66" />
-    </joint>
     <!-- 撼地者 -->
-    <xacro:include filename="$(find hdz_simplified)/urdf/hdz_simplified.xacro" />
-    <joint name="hdz_joint" type="fixed">
-        <parent link="robot_base" />
-        <child link="hdz_base_link" />
-        <origin xyz="0.0 0.0 0.0" rpy="0.0 0.0 0.0" />
-    </joint>
-    <!-- UR model -->
-    <xacro:arg name="ur_parent" default="hdz_ur_base_link" />
+    <xacro:arg name="hdz_tf_prefix" default="hdz_" />
+    <xacro:include filename="$(find ur_perception_description)/urdf/hdz.urdf.xacro" />
+    <!-- UR arm -->
+    <xacro:arg name="ur_parent" default="$(arg hdz_tf_prefix)ur_base_link" />
     <xacro:include filename="$(find ur_perception_description)/urdf/ur5e.urdf.xacro" />
-    <!-- d435i model -->
-    <xacro:arg name="use_nominal_extrinsics" default="false" />
-    <xacro:include filename="$(find realsense2_description)/urdf/_d435i.urdf.xacro" />
-    <xacro:sensor_d435i parent="base"
-        use_nominal_extrinsics="$(arg use_nominal_extrinsics)">
-        <origin xyz="0.0 0.0 2" rpy="0.0 ${pi/2} 0.0" />
-    </xacro:sensor_d435i>
-    <!-- gazebo camera -->
-    <joint name="camera_optical_joint" type="fixed">
-        <origin xyz="0 0 0" rpy="${-pi/2} 0 ${-pi/2}" />
-        <parent link="camera_link" />
-        <child link="camera_link_optical" />
-    </joint>
-    <link name="camera_link_optical"></link>
-    <!-- Add a gazebo tag for the ORIGINAL camera_link (but in the plugin we reference the optical
-    frame so that ROS can orient things correctly) -->
-    <!-- Within the gazebo tag we have the sensor tag, and inside that there is (among other things)
-    the camera tag with the camera parameters, and the plugin tag with some extra parameters the
-    plugin needs. -->
-    <!-- Note that although visualise is set to true, it won't actually visualise the depth camera
-    in gazebo. To see the preview, try swapping "depth" to "camera"-->
-    <gazebo reference="camera_link">
-        <sensor type="depth" name="my_camera">
-            <update_rate>20</update_rate>
-            <visualize>true</visualize>
-            <camera name="cam">
-                <horizontal_fov>1.3962634</horizontal_fov>
-                <image>
-                    <width>640</width>
-                    <height>480</height>
-                    <format>R8G8B8</format>
-                </image>
-                <clip>
-                    <near>0.02</near>
-                    <far>300</far>
-                </clip>
-                <noise>
-                    <type>gaussian</type>
-                    <mean>0.0</mean>
-                    <stddev>0.007</stddev>
-                </noise>
-            </camera>
-            <plugin name="camera_controller" filename="libgazebo_ros_camera.so">
-                <frame_name>camera_link_optical</frame_name>
-                <min_depth>0.1</min_depth>
-                <max_depth>500</max_depth>
-            </plugin>
-        </sensor>
-    </gazebo>
+    <!-- d435i depth camera -->
+    <xacro:include filename="$(find ur_perception_description)/urdf/d435i.xacro" />
 </robot>

File: ur_perception_description/urdf/ur5e.urdf.xacro (robot description, xacro)
@@ -11,9 +11,7 @@
   <xacro:arg name="safety_k_position" default="20" />
   <!-- ros2_control related parameters -->
-  <xacro:arg name="robot_ip" default="0.0.0.0" />
-  <xacro:arg name="reverse_ip" default="0.0.0.0" />
+  <xacro:arg name="ur_robot_ip" default="0.0.0.0" />
+  <xacro:arg name="ur_reverse_ip" default="0.0.0.0" />
   <!-- Simulation parameters -->
-  <xacro:arg name="use_fake_hardware" default="false" />
-  <xacro:arg name="fake_sensor_commands" default="false" />
   <xacro:arg name="sim_gazebo" default="false" />
   <xacro:arg name="sim_ignition" default="false" />
@@ -37,6 +35,6 @@
     safety_pos_margin="$(arg safety_pos_margin)"
     safety_k_position="$(arg safety_k_position)"
-    use_fake_hardware="$(arg use_fake_hardware)"
-    fake_sensor_commands="$(arg fake_sensor_commands)"
+    use_fake_hardware="false"
+    fake_sensor_commands="false"
     sim_gazebo="$(arg sim_gazebo)"
     sim_ignition="$(arg sim_ignition)"
@@ -52,9 +50,9 @@
     tool_device_name="/tmp/ttyUR"
     tool_tcp_port="54321"
-    robot_ip="$(arg robot_ip)"
+    robot_ip="$(arg ur_robot_ip)"
     script_filename=""
     output_recipe_filename=""
     input_recipe_filename=""
-    reverse_ip="$(arg reverse_ip)"
+    reverse_ip="$(arg ur_reverse_ip)"
     script_command_port="50004"
     reverse_port="50001"
