Commit message: successfully controlled real robot

File: hdz_simplified/urdf/hdz_simplified_macro.xacro (robot description, xacro)
@@ -106,5 +106,5 @@
             <origin
                 xyz="0.13075 0 -0.09"
-                rpy="0 0 0" />
+                rpy="0 0 ${pi}" />
             <parent
                 link="${tf_prefix}extend_board_link" />

File: ur_perception_description/srdf/ur_macro.srdf.xacro (robot description, xacro)
@@ -30,26 +30,26 @@
     STATES - Purpose - Define a named state for a particular group, in terms of joint values. This
     is useful to define states like 'folded arms'-->
-    <group_state name="${prefix}home" group="${prefix}ur_manipulator">
-      <joint name="${prefix}elbow_joint" value="0" />
-      <joint name="${prefix}shoulder_lift_joint" value="-1.5707" />
-      <joint name="${prefix}shoulder_pan_joint" value="0" />
-      <joint name="${prefix}wrist_1_joint" value="0" />
-      <joint name="${prefix}wrist_2_joint" value="0" />
-      <joint name="${prefix}wrist_3_joint" value="0" />
-    </group_state>
     <group_state name="${prefix}up" group="${prefix}ur_manipulator">
-      <joint name="${prefix}elbow_joint" value="0" />
-      <joint name="${prefix}shoulder_lift_joint" value="-1.5707" />
-      <joint name="${prefix}shoulder_pan_joint" value="0" />
-      <joint name="${prefix}wrist_1_joint" value="-1.5707" />
-      <joint name="${prefix}wrist_2_joint" value="0" />
-      <joint name="${prefix}wrist_3_joint" value="0" />
+      <joint name="shoulder_pan_joint" value="${pi}" />
+      <joint name="shoulder_lift_joint" value="${-pi/2}" />
+      <joint name="elbow_joint" value="0" />
+      <joint name="wrist_1_joint" value="0" />
+      <joint name="wrist_2_joint" value="0" />
+      <joint name="wrist_3_joint" value="0" />
     </group_state>
     <group_state name="fold" group="${prefix}ur_manipulator">
-      <joint name="elbow_joint" value="2.7317" />
-      <joint name="shoulder_lift_joint" value="-2.6635" />
-      <joint name="shoulder_pan_joint" value="0.2049" />
-      <joint name="wrist_1_joint" value="-3.14" />
-      <joint name="wrist_2_joint" value="-1.57" />
+      <joint name="elbow_joint" value="2.706" />
+      <joint name="shoulder_lift_joint" value="-2.507" />
+      <joint name="shoulder_pan_joint" value="3.414" />
+      <joint name="wrist_1_joint" value="-2.538" />
+      <joint name="wrist_2_joint" value="-1.674" />
+      <joint name="wrist_3_joint" value="0" />
+    </group_state>
+    <group_state name="home" group="${prefix}ur_manipulator">
+      <joint name="shoulder_pan_joint" value="${pi}" />
+      <joint name="shoulder_lift_joint" value="${-pi/2}" />
+      <joint name="elbow_joint" value="${pi/2}" />
+      <joint name="wrist_1_joint" value="${-pi/2}" />
+      <joint name="wrist_2_joint" value="${-pi/2}" />
       <joint name="wrist_3_joint" value="0" />
     </group_state>

File: ur_perception_description/urdf/hdz.urdf.xacro (robot description, xacro)
@@ -3,5 +3,5 @@
     <xacro:include filename="$(find hdz_simplified)/urdf/hdz_simplified_macro.xacro" />
     <xacro:hdz_simplified parent="world" tf_prefix="$(arg hdz_tf_prefix)">
-        <origin xyz="0.0 0.62 0.19" rpy="0.0 0.0 -1.66" />  <!-- 撼地者的位置 -->
+        <origin xyz="0.0 0.0 0.0" rpy="0.0 0.0 0.0" />  <!-- 撼地者的位置 -->
     </xacro:hdz_simplified>
 </robot>
