Commit message: Update sensor and camera positions in urdf file

File: ur_perception_description/urdf/ue5e_perception.urdf.xacro (robot description, xacro)
@@ -8,9 +8,9 @@
     <xacro:sensor_d435i parent="base"
         use_nominal_extrinsics="$(arg use_nominal_extrinsics)">
-        <origin xyz="-0.5 0.0 1.0" rpy="0.0 ${pi/4} 0.0" />
+        <origin xyz="0 0.0 2.0" rpy="0.0 ${pi/2} 0.0" />
     </xacro:sensor_d435i>
     <!-- gazebo camera -->
     <joint name="camera_optical_joint" type="fixed">
-        <origin xyz="0 0 0" rpy="-1.571 0 -1.571" />
+        <origin xyz="0 0 0" rpy="${-pi/2} 0 ${-pi/2}" />
         <parent link="camera_link" />
         <child link="camera_link_optical" />

Commit message: Update sensor position and octomap resolution

File: ur_perception_description/urdf/ue5e_perception.urdf.xacro (robot description, xacro)
@@ -8,5 +8,5 @@
     <xacro:sensor_d435i parent="base"
         use_nominal_extrinsics="$(arg use_nominal_extrinsics)">
-        <origin xyz="0 0.0 2.0" rpy="0.0 ${pi/2} 0.0" />
+        <origin xyz="0.0 0.0 1.5" rpy="0.0 ${pi/2} 0.0" />
     </xacro:sensor_d435i>
     <!-- gazebo camera -->

Commit message: add 撼地者 simplified description

File: ur_perception_description/urdf/ue5e_perception.urdf.xacro (robot description, xacro)
@@ -8,5 +8,5 @@
     <xacro:sensor_d435i parent="base"
         use_nominal_extrinsics="$(arg use_nominal_extrinsics)">
-        <origin xyz="0.0 0.0 1.5" rpy="0.0 ${pi/2} 0.0" />
+        <origin xyz="0.0 0.0 2" rpy="0.0 ${pi/2} 0.0" />
     </xacro:sensor_d435i>
     <!-- gazebo camera -->

Commit message: add robotiq

File: ur_perception_description/urdf/ue5e_perception.urdf.xacro (robot description, xacro)
@@ -13,4 +13,9 @@
     <xacro:arg name="ur_parent" default="hdz_up_board" />
     <xacro:include filename="$(find ur_perception_description)/urdf/ur5e.urdf.xacro" />
+    <!-- RobotIQ Gripper -->
+    <xacro:include filename="$(find robotiq)/urdf/robotiq_85_gripper.urdf.xacro" />
+    <xacro:robotiq_85_gripper prefix="" parent="tool0">
+        <origin xyz="0 0 0" rpy="0 0 0" />
+    </xacro:robotiq_85_gripper>
     <!-- d435i model -->
     <xacro:arg name="use_nominal_extrinsics" default="false" />

Commit message: 添加夹爪

File: ur_perception_description/urdf/ue5e_perception.urdf.xacro (robot description, xacro)
@@ -14,8 +14,60 @@
     <xacro:include filename="$(find ur_perception_description)/urdf/ur5e.urdf.xacro" />
     <!-- RobotIQ Gripper -->
-    <xacro:include filename="$(find robotiq)/urdf/robotiq_85_gripper.urdf.xacro" />
-    <xacro:robotiq_85_gripper prefix="" parent="tool0">
+    <xacro:include filename="$(find robotiq_description)/urdf/robotiq_2f_85_macro.urdf.xacro" />
+    <xacro:robotiq_gripper name="RobotiqGripperHardwareInterface" prefix="" parent="tool0"
+        use_fake_hardware="true">
         <origin xyz="0 0 0" rpy="0 0 0" />
-    </xacro:robotiq_85_gripper>
+    </xacro:robotiq_gripper>
+    <ros2_control name="RobotIQGazeboSystem" type="system">
+        <hardware>
+            <plugin>gazebo_ros2_control/GazeboSystem</plugin>
+        </hardware>
+        <joint name="robotiq_85_left_knuckle_joint">
+            <command_interface name="position" />
+            <state_interface name="position" />
+            <state_interface name="velocity" />
+            <state_interface name="effort" />
+        </joint>
+        <joint name="robotiq_85_right_knuckle_joint">
+            <!-- <param name="mimic">robotiq_85_left_knuckle_joint</param>
+            <param name="multiplier">-1</param> -->
+            <command_interface name="position" />
+            <state_interface name="position" />
+            <state_interface name="velocity" />
+            <state_interface name="effort" />
+        </joint>
+        <joint name="robotiq_85_left_inner_knuckle_joint">
+            <!-- <param name="mimic">robotiq_85_left_knuckle_joint</param>
+            <param name="multiplier">1</param> -->
+            <command_interface name="position" />
+            <state_interface name="position" />
+            <state_interface name="velocity" />
+            <state_interface name="effort" />
+        </joint>
+        <joint name="robotiq_85_right_inner_knuckle_joint">
+            <!-- <param name="mimic">robotiq_85_left_knuckle_joint</param>
+            <param name="multiplier">-1</param> -->
+            <command_interface name="position" />
+            <state_interface name="position" />
+            <state_interface name="velocity" />
+            <state_interface name="effort" />
+        </joint>
+        <joint name="robotiq_85_left_finger_tip_joint">
+            <!-- <param name="mimic">robotiq_85_left_knuckle_joint</param>
+            <param name="multiplier">-1</param> -->
+            <command_interface name="position" />
+            <state_interface name="position" />
+            <state_interface name="velocity" />
+            <state_interface name="effort" />
+        </joint>
+        <joint name="robotiq_85_right_finger_tip_joint">
+            <!-- <param name="mimic">robotiq_85_left_knuckle_joint</param>
+            <param name="multiplier">1</param> -->
+            <command_interface name="position" />
+            <state_interface name="position" />
+            <state_interface name="velocity" />
+            <state_interface name="effort" />
+        </joint>
+    </ros2_control>
     <!-- d435i model -->
     <xacro:arg name="use_nominal_extrinsics" default="false" />

Commit message: fix dependency problem; place ur to chassis

File: ur_perception_description/urdf/ue5e_perception.urdf.xacro (robot description, xacro)
@@ -4,12 +4,12 @@
     <link name="world" />
     <!-- 撼地者 -->
-    <xacro:include filename="$(find hdz_simplified)/urdf/hdz_simplified.urdf" />
+    <xacro:include filename="$(find hdz_simplified)/urdf/hdz_simplified.xacro" />
     <joint name="hdz_joint" type="fixed">
         <parent link="world" />
-        <child link="hdz_up_board" />
-        <origin xyz="0.0 0.0 0.487" rpy="0.0 0.0 0.0" />
+        <child link="hdz_base_link" />
+        <origin xyz="0.0 0.0 0.0" rpy="0.0 0.0 0.0" />
     </joint>
     <!-- UR model -->
-    <xacro:arg name="ur_parent" default="hdz_up_board" />
+    <xacro:arg name="ur_parent" default="hdz_arm_base_link" />
     <xacro:include filename="$(find ur_perception_description)/urdf/ur5e.urdf.xacro" />
     <!-- RobotIQ Gripper -->

File: ur_perception_description/urdf/ur5e.urdf.xacro (robot description, xacro)
@@ -87,5 +87,5 @@
      trajectory_port="$(arg trajectory_port)"
      >
-     <origin xyz="0 -0.3 0.03" rpy="0 0 0" />          <!-- position robot in the world -->
+     <origin xyz="0 0 0" rpy="0 0 0" />          <!-- position robot in the world -->
    </xacro:ur_robot>
    <xacro:if value="$(arg sim_gazebo)">

Commit message: add gaaebo world back

File: ur_perception_description/urdf/ue5e_perception.urdf.xacro (robot description, xacro)
@@ -7,5 +7,5 @@
         <parent link="world" />
         <child link="robot_base" />
-        <origin xyz="0.0 0.0 0.0" rpy="0.0 0.0 0.0" />
+        <origin xyz="0.0 0.62 0.19" rpy="0.0 0.0 -1.66" />
     </joint>
     <!-- 撼地者 -->
