Commit message: add dh_ag95_gripper urdf

File: ur_perception_description/urdf/hdz_with_ur.urdf.xacro (robot description, xacro)
@@ -10,5 +10,7 @@
     <xacro:include filename="$(find ur_perception_description)/urdf/ur5e.urdf.xacro" />
     <!-- RobotIQ Gripper -->
-    <xacro:include filename="$(find ur_perception_description)/urdf/robotiq.urdf.xacro" />
+    <!-- <xacro:include filename="$(find ur_perception_description)/urdf/robotiq.xacro" /> -->
+    <!-- DH Robotics AG95 Gripper -->
+    <xacro:include filename="$(find ur_perception_description)/urdf/dh_ag95_gripper.xacro" />
     <!-- d435i depth camera -->
     <xacro:include filename="$(find ur_perception_description)/urdf/d435i.xacro" />

File: ur_perception_description/urdf/robotiq.xacro (robot description, xacro)
@@ -2,4 +2,9 @@
 <robot xmlns:xacro="http://www.ros.org/wiki/xacro">
     <xacro:include filename="$(find robotiq_description)/urdf/ur_to_robotiq_adapter.urdf.xacro" />
-    <xacro:ur_to_robotiq parent="tool0" />
+    <xacro:ur_to_robotiq prefix="" connected_to="tool0" />
+    <xacro:include filename="$(find robotiq_description)/urdf/robotiq_2f_85_macro.urdf.xacro" />
+    <xacro:robotiq_gripper name="RobotiqGripperHardwareInterface" prefix=""
+        parent="gripper_mount_link" use_fake_hardware="$(arg use_fake_hardware)">
+        <origin xyz="0 0 0" rpy="0 0 0" />
+    </xacro:robotiq_gripper>
 </robot>
