Commit message: fix d435i in gazebo

File: ur_perception_description/urdf/d435i.xacro (robot description, xacro)
@@ -2,4 +2,5 @@
 <robot xmlns:xacro="http://www.ros.org/wiki/xacro">
     <xacro:arg name="use_nominal_extrinsics" default="false" />
+    <xacro:arg name="sim_gazebo" default="false" />
     <!-- d435i depth camera -->
     <xacro:include filename="$(find realsense2_description)/urdf/_d435i.urdf.xacro" />
@@ -7,3 +8,10 @@
         <origin xyz="-0.00235193 -0.06200663  0.02117095" rpy="-2.33887904 -1.56538734 -2.34484763" />
     </xacro:sensor_d435i>
+    <xacro:if value="$(arg sim_gazebo)">
+        <xacro:include filename="$(find ur_perception_description)/urdf/gazebo_rgbd.xacro" />
+        <xacro:gazebo_camera parent="tool0">
+            <origin xyz="-0.0345040364877853 -0.0759815185860376 0.03063655608100728"
+                rpy="${0.00336741+pi/2} ${-0.01153856-pi/2}  0.02297956" />
+        </xacro:gazebo_camera>
+    </xacro:if>
 </robot>

File: ur_perception_description/urdf/gazebo_rgbd.xacro (robot description, xacro)
@@ -1,45 +1,57 @@
 <?xml version="1.0"?>
 <robot xmlns:xacro="http://www.ros.org/wiki/xacro">
-    <!-- gazebo camera -->
-    <joint name="gazebo_camera_optical_joint" type="fixed">
-        <origin xyz="0 0 0" rpy="${-pi/2} 0 ${-pi/2}" />
-        <parent link="camera_link" />
-        <child link="gazebo_camera_link_optical" />
-    </joint>
-    <link name="gazebo_camera_link_optical"></link>
-    <!-- Add a gazebo tag for the ORIGINAL camera_link (but in the plugin we reference the optical
-    frame so that ROS can orient things correctly) -->
-    <!-- Within the gazebo tag we have the sensor tag, and inside that there is (among other things)
-    the camera tag with the camera parameters, and the plugin tag with some extra parameters the
-    plugin needs. -->
-    <!-- Note that although visualise is set to true, it won't actually visualise the depth camera
-    in gazebo. To see the preview, try swapping "depth" to "camera"-->
-    <gazebo reference="camera_link">
-        <sensor type="depth" name="gazebo_camera">
-            <update_rate>20</update_rate>
-            <visualize>true</visualize>
-            <camera name="gz_cam">
-                <horizontal_fov>1.3962634</horizontal_fov>
-                <image>
-                    <width>640</width>
-                    <height>480</height>
-                    <format>R8G8B8</format>
-                </image>
-                <clip>
-                    <near>0.02</near>
-                    <far>300</far>
-                </clip>
-                <noise>
-                    <type>gaussian</type>
-                    <mean>0.0</mean>
-                    <stddev>0.007</stddev>
-                </noise>
-            </camera>
-            <plugin name="camera_controller" filename="libgazebo_ros_camera.so">
-                <frame_name>gazebo_camera_link_optical</frame_name>
-                <min_depth>0.1</min_depth>
-                <max_depth>500</max_depth>
-            </plugin>
-        </sensor>
-    </gazebo>
+    <xacro:macro name="gazebo_camera" params="parent prefix:=gazebo_ *origin">
+        <!-- gazebo camera link -->
+        <link name="${prefix}camera_link"></link>
+        <joint name="${prefix}camera_joint" type="fixed">
+            <xacro:insert_block name="origin" />
+            <parent link="${parent}" />
+            <child link="${prefix}camera_link" />
+        </joint>
+        <!-- gazebo camera optical link(frame) -->
+        <link name="${prefix}camera_optical_link"></link>
+        <joint name="${prefix}camera_optical_joint" type="fixed">
+            <origin xyz="0 0 0" rpy="${-pi/2} 0 ${-pi/2}" />
+            <parent link="${prefix}camera_link" />
+            <child link="${prefix}camera_optical_link" />
+        </joint>
+        <!-- Add a gazebo tag for the ORIGINAL camera_link (but in the plugin we reference optical
+        frame so that ROS can orient things correctly) -->
+        <!-- Within the gazebo tag we have the sensor tag, and inside that there is (among other
+        things)
+    the camera tag with the camera parameters, and the plugin tag with some extra parameters the plugin
+        needs. -->
+        <!-- Note that although visualise is set to true, it won't actually visualise the depth
+        camera in gazebo. To see the preview, try swapping "depth" to "camera"-->
+        <gazebo reference="${prefix}camera_link">
+            <sensor type="depth" name="camera">
+                <update_rate>20</update_rate>
+                <visualize>true</visualize>
+                <camera name="gz_cam">
+                    <horizontal_fov>1.3962634</horizontal_fov>
+                    <image>
+                        <width>640</width>
+                        <height>480</height>
+                        <format>R8G8B8</format>
+                    </image>
+                    <clip>
+                        <near>0.02</near>
+                        <far>300</far>
+                    </clip>
+                    <noise>
+                        <type>gaussian</type>
+                        <mean>0.0</mean>
+                        <stddev>0.007</stddev>
+                    </noise>
+                </camera>
+                <plugin name="camera_controller" filename="libgazebo_ros_camera.so">
+                    <frame_name>${prefix}camera_optical_link</frame_name>
+                    <namespace>camera/depth</namespace>
+                    <camera_name>color</camera_name>
+                    <min_depth>0.1</min_depth>
+                    <max_depth>500</max_depth>
+                </plugin>
+            </sensor>
+        </gazebo>
+    </xacro:macro>
 </robot>

Commit message: move_grasp添加坐标转换功能

File: ur_perception_description/urdf/d435i.xacro (robot description, xacro)
@@ -10,5 +10,5 @@
     <xacro:if value="$(arg sim_gazebo)">
         <xacro:include filename="$(find ur_perception_description)/urdf/gazebo_rgbd.xacro" />
-        <xacro:gazebo_camera parent="tool0">
+        <xacro:gazebo_camera parent="tool0" camera_link_name="gazebo_camera_link">
             <origin xyz="-0.0345040364877853 -0.0759815185860376 0.03063655608100728"
                 rpy="${0.00336741+pi/2} ${-0.01153856-pi/2}  0.02297956" />

File: ur_perception_description/urdf/gazebo_rgbd.xacro (robot description, xacro)
@@ -1,18 +1,18 @@
 <?xml version="1.0"?>
 <robot xmlns:xacro="http://www.ros.org/wiki/xacro">
-    <xacro:macro name="gazebo_camera" params="parent prefix:=gazebo_ *origin">
+    <xacro:macro name="gazebo_camera" params="parent camera_link_name:=camera_link optical_link_name:=camera_color_optical_frame *origin">
         <!-- gazebo camera link -->
-        <link name="${prefix}camera_link"></link>
-        <joint name="${prefix}camera_joint" type="fixed">
+        <link name="${camera_link_name}"></link>
+        <joint name="${camera_link_name}_joint" type="fixed">
             <xacro:insert_block name="origin" />
             <parent link="${parent}" />
-            <child link="${prefix}camera_link" />
+            <child link="${camera_link_name}" />
         </joint>
         <!-- gazebo camera optical link(frame) -->
-        <link name="${prefix}camera_optical_link"></link>
-        <joint name="${prefix}camera_optical_joint" type="fixed">
+        <link name="${optical_link_name}"></link>
+        <joint name="${optical_link_name}_joint" type="fixed">
             <origin xyz="0 0 0" rpy="${-pi/2} 0 ${-pi/2}" />
-            <parent link="${prefix}camera_link" />
-            <child link="${prefix}camera_optical_link" />
+            <parent link="${camera_link_name}" />
+            <child link="${optical_link_name}" />
         </joint>
         <!-- Add a gazebo tag for the ORIGINAL camera_link (but in the plugin we reference optical
@@ -24,5 +24,5 @@
         <!-- Note that although visualise is set to true, it won't actually visualise the depth
         camera in gazebo. To see the preview, try swapping "depth" to "camera"-->
-        <gazebo reference="${prefix}camera_link">
+        <gazebo reference="${camera_link_name}">
             <sensor type="depth" name="camera">
                 <update_rate>20</update_rate>
@@ -46,5 +46,5 @@
                 </camera>
                 <plugin name="camera_controller" filename="libgazebo_ros_camera.so">
-                    <frame_name>${prefix}camera_optical_link</frame_name>
+                    <frame_name>${optical_link_name}</frame_name>
                     <namespace>camera/depth</namespace>
                     <camera_name>color</camera_name>
