Commit message: add gripper in gazebo

File: dh_robotics_ag95_description/urdf/dh_robotics_ag95_gripper.urdf.xacro (robot description, xacro)
@@ -1,5 +1,8 @@
 <?xml version="1.0"?>
 <robot name="dh_robotics_ag95_gripper" xmlns:xacro="http://ros.org/wiki/xacro">
-    <!-- <xacro:include filename="$(find dh_robotics_ag95_description)/urdf/dh_robotics_ag95_gripper.transmission.xacro" /> -->
+    <!-- <xacro:include filename="$(find
+    dh_robotics_ag95_description)/urdf/dh_robotics_ag95_gripper.transmission.xacro" /> -->
+    <xacro:include
+        filename="$(find dh_robotics_ag95_description)/urdf/dh_robotics_ag95_gripper_ros2_control.xacro" />
     <xacro:macro name="material_black">
         <material name="">
@@ -361,4 +364,5 @@
         </gazebo>
         <!-- <xacro:dh_robotics_ag95_gripper_transmission prefix="${prefix}" /> -->
+        <xacro:dh_robotics_ag95_gripper_ros2_control prefix="${prefix}" />
     </xacro:macro>
 </robot>

File: dh_robotics_ag95_description/urdf/dh_robotics_ag95_gripper.xacro (robot description, xacro)
@@ -1,28 +1,23 @@
-<?xml version="1.0" ?>
+<?xml version="1.0"?>
 <robot name="dh_robotics_ag95_gripper" xmlns:xacro="http://ros.org/wiki/xacro">
-    <xacro:include filename="$(find dh_robotics_ag95_description)/urdf/dh_robotics_ag95_gripper.urdf.xacro" />
-    <gazebo>
-        <plugin name="gazebo_ros_control" filename="libgazebo_ros_control.so">
-            <robotNamespace>/</robotNamespace>
-            <legacyModeNS>true</legacyModeNS>
-        </plugin>
-    </gazebo>
-    <link name="world"/>
+    <xacro:include
+        filename="$(find dh_robotics_ag95_description)/urdf/dh_robotics_ag95_gripper.urdf.xacro" />
+    <link name="world" />
     <joint name="world_fixed" type="fixed">
-        <origin xyz="0 0 0" rpy="0 0 0"/>
-        <parent link="world"/>
-        <child link="gripper_root_link"/>
+        <origin xyz="0 0 0" rpy="0 0 0" />
+        <parent link="world" />
+        <child link="gripper_root_link" />
     </joint>
     <link name="gripper_root_link">
         <visual>
-            <origin xyz="0 0 0.5" rpy="0 0 0"/>
+            <origin xyz="0 0 0.5" rpy="0 0 0" />
             <geometry>
-                <box size="0.1 0.1 1.0"/>
+                <box size="0.1 0.1 1.0" />
             </geometry>
         </visual>
         <collision>
-            <origin xyz="0 0 0.5" rpy="0 0 0"/>
+            <origin xyz="0 0 0.5" rpy="0 0 0" />
             <geometry>
-                <box size="0.1 0.1 1.0"/>
+                <box size="0.1 0.1 1.0" />
             </geometry>
         </collision>
@@ -30,11 +25,19 @@
             <mass value="1e2" />
             <origin xyz="0.0 0.0 0.0" />
-            <inertia ixx = "0.000001" ixy = "0.000000" ixz = "0.000000"
-                     iyx = "0.000000" iyy = "0.000001" iyz = "0.000000"
-                     izx = "0.000000" izy = "0.000000" izz = "0.000001" />
+            <inertia ixx="0.000001" ixy="0.000000" ixz="0.000000"
+                iyx="0.000000" iyy="0.000001" iyz="0.000000"
+                izx="0.000000" izy="0.000000" izz="0.000001" />
         </inertial>
     </link>
-    <xacro:dh_robotics_ag95_gripper prefix="" parent="gripper_root_link" >
-        <origin xyz="0.05 0 0.85" rpy="${pi/2}  0 ${pi/2}"/>
+    <xacro:dh_robotics_ag95_gripper prefix="" parent="gripper_root_link">
+        <origin xyz="0.05 0 0.85" rpy="${pi/2}  0 ${pi/2}" />
     </xacro:dh_robotics_ag95_gripper>
+    <gazebo>
+        <plugin filename="libgazebo_ros2_control.so" name="dh_gazebo_ros2_control">
+            <!-- <robot_param>robot_description</robot_param>
+            <robot_param_node>robot_state_publisher</robot_param_node> -->
+            <parameters>$(find dh_robotics_ag95_description)/config/dh_controllers.yaml</parameters>
+            <!-- <controller_manager_name>controller_manager</controller_manager_name> -->
+        </plugin>
+    </gazebo>
 </robot>

Commit message: handeye calibration; d435 with moveit

File: dh_robotics_ag95_description/urdf/dh_robotics_ag95_gripper.urdf.xacro (robot description, xacro)
@@ -364,5 +364,6 @@
         </gazebo>
         <!-- <xacro:dh_robotics_ag95_gripper_transmission prefix="${prefix}" /> -->
-        <xacro:dh_robotics_ag95_gripper_ros2_control prefix="${prefix}" />
+        <xacro:arg name="sim_gazebo" default="false" />
+        <xacro:dh_robotics_ag95_gripper_ros2_control prefix="${prefix}" sim_gazebo="$(arg sim_gazebo)" />
     </xacro:macro>
 </robot>

File: dh_robotics_ag95_description/urdf/dh_robotics_ag95_gripper_ros2_control.xacro (robot description, xacro)
@@ -1,69 +1,71 @@
 <?xml version="1.0"?>
 <robot xmlns:xacro="http://ros.org/wiki/xacro">
-    <xacro:macro name="dh_robotics_ag95_gripper_ros2_control" params="prefix">
-        <ros2_control name="ag95_gripper" type="system">
-            <hardware>
-                <plugin>gazebo_ros2_control/GazeboSystem</plugin>
-            </hardware>
-            <joint name="${prefix}gripper_finger1_joint">
-                <command_interface name="position">
-                    <param name="min">0.0</param>
-                    <param name="max">0.65</param>
-                </command_interface>
-                <state_interface name="position">
-                    <param name="initial_value">0.0</param>
-                </state_interface>
-                <state_interface name="velocity" />
-                <state_interface name="effort" />
-            </joint>
-            <joint name="${prefix}gripper_finger2_joint">
-                <param name="mimic">${prefix}gripper_finger1_joint</param>
-                <state_interface name="position" />
-                <state_interface name="velocity" />
-                <state_interface name="effort" />
-            </joint>
-            <joint name="${prefix}gripper_finger1_finger_joint">
-                <param name="mimic">${prefix}gripper_finger1_joint</param>
-                <param name="multiplier">0.4563942</param>
-                <state_interface name="position" />
-                <state_interface name="velocity" />
-                <state_interface name="effort" />
-            </joint>
-            <joint name="${prefix}gripper_finger2_finger_joint">
-                <param name="mimic">${prefix}gripper_finger1_joint</param>
-                <param name="multiplier">0.4563942</param>
-                <state_interface name="position" />
-                <state_interface name="velocity" />
-                <state_interface name="effort" />
-            </joint>
-            <joint name="${prefix}gripper_finger1_inner_knuckle_joint">
-                <param name="mimic">${prefix}gripper_finger1_joint</param>
-                <param name="multiplier">1.49462955</param>
-                <state_interface name="position" />
-                <state_interface name="velocity" />
-                <state_interface name="effort" />
-            </joint>
-            <joint name="${prefix}gripper_finger2_inner_knuckle_joint">
-                <param name="mimic">${prefix}gripper_finger1_joint</param>
-                <param name="multiplier">1.49462955</param>
-                <state_interface name="position" />
-                <state_interface name="velocity" />
-                <state_interface name="effort" />
-            </joint>
-            <joint name="${prefix}gripper_finger1_finger_tip_joint">
-                <param name="mimic">${prefix}gripper_finger1_joint</param>
-                <param name="multiplier">1.49462955</param>
-                <state_interface name="position" />
-                <state_interface name="velocity" />
-                <state_interface name="effort" />
-            </joint>
-            <joint name="${prefix}gripper_finger2_finger_tip_joint">
-                <param name="mimic">${prefix}gripper_finger1_joint</param>
-                <param name="multiplier">1.49462955</param>
-                <state_interface name="position" />
-                <state_interface name="velocity" />
-                <state_interface name="effort" />
-            </joint>
-        </ros2_control>
+    <xacro:macro name="dh_robotics_ag95_gripper_ros2_control" params="prefix sim_gazebo:=false">
+        <xacro:if value="${sim_gazebo}">
+            <ros2_control name="ag95_gripper" type="system">
+                <hardware>
+                    <plugin>gazebo_ros2_control/GazeboSystem</plugin>
+                </hardware>
+                <joint name="${prefix}gripper_finger1_joint">
+                    <command_interface name="position">
+                        <param name="min">0.0</param>
+                        <param name="max">0.65</param>
+                    </command_interface>
+                    <state_interface name="position">
+                        <param name="initial_value">0.0</param>
+                    </state_interface>
+                    <state_interface name="velocity" />
+                    <state_interface name="effort" />
+                </joint>
+                <joint name="${prefix}gripper_finger2_joint">
+                    <param name="mimic">${prefix}gripper_finger1_joint</param>
+                    <state_interface name="position" />
+                    <state_interface name="velocity" />
+                    <state_interface name="effort" />
+                </joint>
+                <joint name="${prefix}gripper_finger1_finger_joint">
+                    <param name="mimic">${prefix}gripper_finger1_joint</param>
+                    <param name="multiplier">0.4563942</param>
+                    <state_interface name="position" />
+                    <state_interface name="velocity" />
+                    <state_interface name="effort" />
+                </joint>
+                <joint name="${prefix}gripper_finger2_finger_joint">
+                    <param name="mimic">${prefix}gripper_finger1_joint</param>
+                    <param name="multiplier">0.4563942</param>
+                    <state_interface name="position" />
+                    <state_interface name="velocity" />
+                    <state_interface name="effort" />
+                </joint>
+                <joint name="${prefix}gripper_finger1_inner_knuckle_joint">
+                    <param name="mimic">${prefix}gripper_finger1_joint</param>
+                    <param name="multiplier">1.49462955</param>
+                    <state_interface name="position" />
+                    <state_interface name="velocity" />
+                    <state_interface name="effort" />
+                </joint>
+                <joint name="${prefix}gripper_finger2_inner_knuckle_joint">
+                    <param name="mimic">${prefix}gripper_finger1_joint</param>
+                    <param name="multiplier">1.49462955</param>
+                    <state_interface name="position" />
+                    <state_interface name="velocity" />
+                    <state_interface name="effort" />
+                </joint>
+                <joint name="${prefix}gripper_finger1_finger_tip_joint">
+                    <param name="mimic">${prefix}gripper_finger1_joint</param>
+                    <param name="multiplier">1.49462955</param>
+                    <state_interface name="position" />
+                    <state_interface name="velocity" />
+                    <state_interface name="effort" />
+                </joint>
+                <joint name="${prefix}gripper_finger2_finger_tip_joint">
+                    <param name="mimic">${prefix}gripper_finger1_joint</param>
+                    <param name="multiplier">1.49462955</param>
+                    <state_interface name="position" />
+                    <state_interface name="velocity" />
+                    <state_interface name="effort" />
+                </joint>
+            </ros2_control>
+        </xacro:if>
     </xacro:macro>
 </robot>

File: ur_perception_description/urdf/d435i.xacro (robot description, xacro)
@@ -4,49 +4,6 @@
     <!-- d435i depth camera -->
     <xacro:include filename="$(find realsense2_description)/urdf/_d435i.urdf.xacro" />
-    <xacro:sensor_d435i parent="base"
-        use_nominal_extrinsics="$(arg use_nominal_extrinsics)">
-        <origin xyz="0.0 0.0 2" rpy="0.0 ${pi/2} 0.0" />
+    <xacro:sensor_d435i parent="tool0" use_nominal_extrinsics="$(arg use_nominal_extrinsics)">
+        <origin xyz="-0.00235193 -0.06200663  0.02117095" rpy="-2.33887904 -1.56538734 -2.34484763" />
     </xacro:sensor_d435i>
-    <!-- gazebo camera -->
-    <joint name="camera_optical_joint" type="fixed">
-        <origin xyz="0 0 0" rpy="${-pi/2} 0 ${-pi/2}" />
-        <parent link="camera_link" />
-        <child link="camera_link_optical" />
-    </joint>
-    <link name="camera_link_optical"></link>
-    <!-- Add a gazebo tag for the ORIGINAL camera_link (but in the plugin we reference the optical
-    frame so that ROS can orient things correctly) -->
-    <!-- Within the gazebo tag we have the sensor tag, and inside that there is (among other things)
-    the camera tag with the camera parameters, and the plugin tag with some extra parameters the
-    plugin needs. -->
-    <!-- Note that although visualise is set to true, it won't actually visualise the depth camera
-    in gazebo. To see the preview, try swapping "depth" to "camera"-->
-    <gazebo reference="camera_link">
-        <sensor type="depth" name="my_camera">
-            <update_rate>20</update_rate>
-            <visualize>true</visualize>
-            <camera name="cam">
-                <horizontal_fov>1.3962634</horizontal_fov>
-                <image>
-                    <width>640</width>
-                    <height>480</height>
-                    <format>R8G8B8</format>
-                </image>
-                <clip>
-                    <near>0.02</near>
-                    <far>300</far>
-                </clip>
-                <noise>
-                    <type>gaussian</type>
-                    <mean>0.0</mean>
-                    <stddev>0.007</stddev>
-                </noise>
-            </camera>
-            <plugin name="camera_controller" filename="libgazebo_ros_camera.so">
-                <frame_name>camera_link_optical</frame_name>
-                <min_depth>0.1</min_depth>
-                <max_depth>500</max_depth>
-            </plugin>
-        </sensor>
-    </gazebo>
 </robot>
