Commit message: 重构 sim_moveit; 删除Universal_Robots_ROS2_Gazebo_simulation, ur_perception_moveit_launcher

File: ur_perception_description/srdf/ur_macro.srdf.xacro (robot description, xacro)
@@ -7,5 +7,5 @@
   are defined
 -->
-  <xacro:macro name="ur_srdf" params="name prefix">
+  <xacro:macro name="ur_srdf" params="prefix">
     <!--GROUPS
     - Representation of a set of joints and links. This can be useful for specifying DOF to plan
@@ -24,5 +24,5 @@
     <!--SUBGROUPS
     - Groups can also be formed by referencing to already defined group names-->
-    <group name="${prefix}${name}_manipulator">
+    <group name="${prefix}ur_manipulator">
       <chain base_link="${prefix}base_link" tip_link="${prefix}tool0" />
     </group>
@@ -30,5 +30,5 @@
     STATES - Purpose - Define a named state for a particular group, in terms of joint values. This
     is useful to define states like 'folded arms'-->
-    <group_state name="${prefix}home" group="${prefix}${name}_manipulator">
+    <group_state name="${prefix}home" group="${prefix}ur_manipulator">
       <joint name="${prefix}elbow_joint" value="0" />
       <joint name="${prefix}shoulder_lift_joint" value="-1.5707" />
@@ -38,5 +38,5 @@
       <joint name="${prefix}wrist_3_joint" value="0" />
     </group_state>
-    <group_state name="${prefix}up" group="${prefix}${name}_manipulator">
+    <group_state name="${prefix}up" group="${prefix}ur_manipulator">
       <joint name="${prefix}elbow_joint" value="0" />
       <joint name="${prefix}shoulder_lift_joint" value="-1.5707" />
@@ -46,5 +46,5 @@
       <joint name="${prefix}wrist_3_joint" value="0" />
     </group_state>
-    <group_state name="fold" group="${prefix}${name}_manipulator">
+    <group_state name="fold" group="${prefix}ur_manipulator">
       <joint name="elbow_joint" value="2.7317" />
       <joint name="shoulder_lift_joint" value="-2.6635" />

File: ur_perception_description/urdf/hdz_with_ur.urdf.xacro (robot description, xacro)
@@ -1,7 +1,7 @@
 <?xml version="1.0" encoding="UTF-8"?>
-<robot name="ur5e_rgbd" xmlns:xacro="http://www.ros.org/wiki/xacro">
+<robot name="hdz_with_ur" xmlns:xacro="http://www.ros.org/wiki/xacro">
     <!-- create link fixed to the "world" -->
     <link name="world" />
-    <!-- 撼地者 -->
+    <!-- 撼地者 (hdz) -->
     <xacro:arg name="hdz_tf_prefix" default="hdz_" />
     <xacro:include filename="$(find ur_perception_description)/urdf/hdz.urdf.xacro" />

File: ur_perception_moveit_config/config/ur5e_rgbd.urdf.xacro (robot description, xacro)
@@ -3,5 +3,5 @@
     <xacro:arg name="moveit_initial_positions_file" default="$(find ur_perception_moveit_config)/config/initial_positions.yaml" />
     <!-- Import ur5e_rgbd urdf file -->
-    <xacro:include filename="$(find ur_perception_description)/urdf/ue5e_perception.urdf.xacro" />
+    <xacro:include filename="$(find ur_perception_description)/urdf/hdz_with_ur.urdf.xacro" />
     <!-- Import control_xacro -->
     <xacro:include filename="ur5e_rgbd.ros2_control.xacro" />

Commit message: 在仿真和真实环境中成功移动到目标位置

File: ur_perception_description/srdf/ur_macro.srdf.xacro (robot description, xacro)
@@ -25,5 +25,5 @@
     - Groups can also be formed by referencing to already defined group names-->
     <group name="${prefix}ur_manipulator">
-      <chain base_link="${prefix}base_link" tip_link="${prefix}tool0" />
+      <chain base_link="${prefix}base_link" tip_link="grasp_center_link" />
     </group>
     <!--GROUP
@@ -52,4 +52,12 @@
       <joint name="wrist_1_joint" value="${-pi/2}" />
       <joint name="wrist_2_joint" value="${-pi/2}" />
+      <joint name="wrist_3_joint" value="0" />
+    </group_state>
+    <group_state name="ready" group="${prefix}ur_manipulator">
+      <joint name="shoulder_pan_joint" value="${pi}" />
+      <joint name="shoulder_lift_joint" value="-1.4395745706609269" />
+      <joint name="elbow_joint" value="1.9782918135272425" />
+      <joint name="wrist_1_joint" value="-2.1096626720824183" />
+      <joint name="wrist_2_joint" value="-1.57185537019838" />
       <joint name="wrist_3_joint" value="0" />
     </group_state>

File: ur_perception_description/urdf/hdz_with_ur.urdf.xacro (robot description, xacro)
@@ -9,4 +9,10 @@
     <xacro:arg name="ur_parent" default="$(arg hdz_tf_prefix)ur_base_link" />
     <xacro:include filename="$(find ur_perception_description)/urdf/ur5e.urdf.xacro" />
+    <link name="grasp_center_link" />
+    <joint name="grasp_center_joint" type="fixed">
+        <parent link="tool0" />
+        <child link="grasp_center_link" />
+        <origin xyz="0 0 0.18" rpy="0 0 0" />
+    </joint>
     <!-- RobotIQ Gripper -->
     <!-- <xacro:include filename="$(find ur_perception_description)/urdf/robotiq.xacro" /> -->
